File: Hardware/U_I_Source/Design/power_supply/power_supply.kicad_pcb (KiCad board)
At the start: 2 copper layers, 85 x 56.1 mm, 69 parts, among them J1 BANANEN_RED, J2 BANANEN_BLACK, J3 CONN_02X10, J4 USB_OTG, Q1 FDD8778, SW1 BOOT, SW2 RESET, U1 LM1117-ADJ, U2 INA180B1, U3 INA180B1, U4 LMV321, U5 INA180B1, U6 LPC1343FBD48, Y1 12MHz/20pF

Commit message: Updated design files of the U_I_Source OpenLab Tool - latest version
Parts:
- removed the C15 at (145.2, 102.6)
- removed the C21 at (76.5, 81.9)
- removed the REF** at (76.2, 55.7)
- removed the REF** at (76.2, 102.9)
- removed the REF** at (153.8, 102.9)
- removed the REF** at (153.9, 64.0)
- added C12: 22n, Capacitors_SMD:C_0603, F.Cu at (114.3, 97.6)
- added C13: 22n, Capacitors_SMD:C_0603, F.Cu at (117.3, 97.6)
- added C17: 22n, Capacitors_SMD:C_0603, F.Cu at (138.4, 99.2)
- added C20: 22n, Capacitors_SMD:C_0603, F.Cu at (139.3, 102.3)
- added C6: 22n(DNI), Capacitors_SMD:C_0603, F.Cu at (93.8, 92.8)
- added C9: 22n(DNI), Capacitors_SMD:C_0603, F.Cu at (96.8, 92.8)
- added R11: 10, Resistors_SMD:R_0805, F.Cu at (117.8, 100.2)
- added R16: 10, Resistors_SMD:R_0805, F.Cu at (136.8, 99.4)
- added R19: 10, Resistors_SMD:R_0805, F.Cu at (142.4, 102.5)
- added R2: 4k7, Resistors_SMD:R_0603, F.Cu at (98.8, 86.6)
- added R30: 10k, Resistors_SMD:R_0805_HandSoldering, F.Cu at (76.5, 81.8)
- added R4: 10, Resistors_SMD:R_0805, F.Cu at (93.5, 95.5)
- added R6: 10, Resistors_SMD:R_0805, F.Cu at (97.5, 95.5)
- added R8: 10, Resistors_SMD:R_0805, F.Cu at (113.8, 100.2)
- added REF**: 1pin, Connectors:1pin, F.Cu at (76.3, 103.5)
- added REF**: 1pin, Connectors:1pin, F.Cu at (76.3, 55.2)
- added REF**: 1pin, Connectors:1pin, F.Cu at (153.6, 63.8)
- added REF**: 1pin, Connectors:1pin, F.Cu at (153.8, 103.5)
- R9: renamed from R5; value 0.1 -> 0.068
- moved R10 35.8 mm to (96.0, 81.1), turned to 90 degrees
- moved D3 9.94 mm to (108.2, 102.6)
- moved R9 6.26 mm to (115.7, 103.2)
- moved U3 4.31 mm to (116.0, 94.1)
- moved R12 3.80 mm to (120.3, 99.2)
- moved C5 3.65 mm to (92.7, 89.1), turned to 270 degrees
- moved R13 3.40 mm to (120.3, 93.8), turned to 270 degrees
- moved R5 3.27 mm to (95.3, 98.4)
- moved C15 2.92 mm to (144.8, 99.6), turned to 270 degrees
- moved C10 2.80 mm to (103.0, 100.5)
- moved C11 2.55 mm to (113.0, 93.5), turned to 90 degrees
- moved U5 1.70 mm to (141.6, 99.6)
- moved U2 0.95 mm to (95.5, 89.7)
- moved C7 0.62 mm to (99.5, 91.3), turned to 270 degrees
- moved R18 0.42 mm to (140.8, 104.9)
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- renumbered C8 to C10, C9 to C11, C10 to C14, C12 to C15, C11 to C16, C13 to C18, C14 to C19, C16 to C21, C17 to C22, C18 to C23, C19 to C24, C20 to C25, C6 to C7, C7 to C8, R6 to R10, R7 to R12, R8 to R13, R9 to R14, R10 to R15, R11 to R17, R12 to R18, R13 to R20, R14 to R21, R15 to R22, R16 to R23, R17 to R24, R18 to R25, R19 to R26, R20 to R27, R21 to R28, R22 to R29, R2 to R3, R3 to R5, R4 to R7
Connections:
- net L2_current renamed DIODE_current
- net USB_5V renamed VCC
- C10 pad 1: Net-(C8-Pad1) -> Net-(C10-Pad1)
- C10 pad 2: Net-(C8-Pad2) -> Net-(C10-Pad2)
- C16 pad 1: Net-(C11-Pad1) -> Net-(C16-Pad1)
- C18 pad 1: Net-(C11-Pad1) -> Net-(C16-Pad1)
- D3 pad 1: Net-(C11-Pad1) -> Net-(D3-Pad1)
- D3 pad 2: Net-(D3-Pad2) -> Net-(C10-Pad1)
- J3 pad 15: Net-(J3-Pad15) -> (no net)
- J3 pad 19: Net-(J3-Pad19) -> (no net)
- J3 pad 3: Net-(J3-Pad3) -> (no net)
- J3 pad 5: Net-(J3-Pad5) -> (no net)
- J4 pad 4: Net-(J4-Pad4) -> (no net)
- L2 pad 2: Net-(C8-Pad1) -> Net-(C10-Pad1)
- Q1 pad 2: Net-(C8-Pad2) -> Net-(C10-Pad2)
- R12 pad 2: Net-(C11-Pad1) -> Net-(C16-Pad1)
- R18 pad 2: Net-(C11-Pad1) -> Net-(C16-Pad1)
- R5 pad 1: Net-(C8-Pad2) -> Net-(C10-Pad2)
- R9 pad 1: Net-(D3-Pad2) -> Net-(C16-Pad1)
- R9 pad 2: Net-(C8-Pad1) -> Net-(D3-Pad1)
- U2 pad 1: Net-(L1-Pad2) -> Net-(C6-Pad1)
- U2 pad 3: Net-(C8-Pad2) -> Net-(C9-Pad1)
- U3 pad 1: Net-(C8-Pad1) -> Net-(C12-Pad1)
- U3 pad 3: Net-(D3-Pad2) -> Net-(C13-Pad1)
- U5 pad 1: Net-(C11-Pad1) -> Net-(C17-Pad1)
- U5 pad 3: Net-(D6-Pad2) -> Net-(C20-Pad1)
- U6 pad 10: Net-(U6-Pad10) -> (no net)
- U6 pad 11: Net-(U6-Pad11) -> (no net)
- U6 pad 12: Net-(U6-Pad12) -> (no net)
- U6 pad 13: Net-(U6-Pad13) -> (no net)
- U6 pad 15: Net-(U6-Pad15) -> (no net)
- U6 pad 16: Net-(U6-Pad16) -> (no net)
- U6 pad 17: Net-(U6-Pad17) -> (no net)
- U6 pad 18: Net-(U6-Pad18) -> (no net)
- U6 pad 21: Net-(U6-Pad21) -> (no net)
- U6 pad 22: USB_CONNECT -> (no net)
- U6 pad 23: Net-(U6-Pad23) -> (no net)
- U6 pad 24: Net-(U6-Pad24) -> (no net)
- U6 pad 25: Net-(U6-Pad25) -> (no net)
- U6 pad 26: Net-(U6-Pad26) -> (no net)
- U6 pad 30: Net-(U6-Pad30) -> (no net)
- U6 pad 31: Net-(U6-Pad31) -> (no net)
- U6 pad 36: Net-(U6-Pad36) -> (no net)
- U6 pad 37: Net-(U6-Pad37) -> (no net)
- U6 pad 38: Net-(U6-Pad38) -> (no net)
- U6 pad 40: Net-(U6-Pad40) -> (no net)
- U6 pad 42: Net-(U6-Pad42) -> (no net)
- U6 pad 43: Net-(U6-Pad43) -> (no net)
- U6 pad 45: Net-(U6-Pad45) -> (no net)
- U6 pad 46: Net-(U6-Pad46) -> (no net)
- U6 pad 47: Net-(U6-Pad47) -> (no net)
- U6 pad 48: Net-(U6-Pad48) -> (no net)
- U6 pad 9: Net-(U6-Pad9) -> (no net)
Routing:
- net GNDA: track 44.6 -> 124.4 mm, vias 4 -> 25
- net GNDD: track 49.1 -> 107.0 mm, vias 8 -> 23
- net Net-(C16-Pad1): track 0.00 -> 35.4 mm
- net Net-(C11-Pad1): track 31.0 -> 0.00 mm
- net Net-(C8-Pad1): track 30.1 -> 0.00 mm
- net Net-(C10-Pad1): track 0.00 -> 28.0 mm
- net Net-(C10-Pad2): track 0.00 -> 24.2 mm
- net Net-(C8-Pad2): track 22.1 -> 0.00 mm
- net 3.3V: track 203.4 -> 224.3 mm
- net Net-(D3-Pad2): track 7.14 -> 0.00 mm
- net Net-(D3-Pad1): track 0.00 -> 6.51 mm
- net load_current: track 70.7 -> 65.9 mm
- net Net-(C13-Pad1): track 0.00 -> 4.48 mm
- net Net-(C12-Pad1): track 0.00 -> 4.36 mm
- net Net-(C6-Pad1): track 0.00 -> 4.18 mm
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Other:
- net class Default: via_dia 0.6 -> 0.7; via_drill 0.4 -> 0.3
- rule pad_to_mask_clearance: 0.2 -> 0
- rule via_min_size: 0.4 -> 0.7
- board text added: "V1.1"
