File: Hardware/U_I_Source/Design/power_supply/power_supply.sch (KiCad schematic (older format))
At the start: 65 parts, among them J1 BANANEN_RED, J2 BANANEN_BLACK, J3 CONN_02X10, J4 USB_OTG, Q1 FDD8778, SW1 BOOT, SW2 RESET, U1 LM1117-ADJ, U2 INA180B1, U3 INA180B1, U4 LMV321, U5 INA180B1, U6 LPC1343FBD48, Y1 12MHz/20pF

Commit message: Updated design files of the U_I_Source OpenLab Tool - latest version
Parts:
- removed C15, C21: 100n, Capacitors_SMD:C_0603_HandSoldering, symbol C
- added C12, C13, C17, C20: 22n, Capacitors_SMD:C_0603, symbol C
- added C6, C9: 22n(DNI), Capacitors_SMD:C_0603, symbol C
- added R11, R16, R19, R4, R6, R8: 10, Resistors_SMD:R_0805, symbol R
- added R2: 4k7, Resistors_SMD:R_0603, symbol R
- added R30: 10k, Resistors_SMD:R_0805_HandSoldering, symbol R
- R9: renamed from R5; value 0.1 -> 0.068
- renumbered C8 to C10, C9 to C11, C10 to C14, C12 to C15, C11 to C16, C13 to C18, C14 to C19, C16 to C21, C17 to C22, C18 to C23, C19 to C24, C20 to C25, C6 to C7, C7 to C8, R6 to R10, R7 to R12, R8 to R13, R9 to R14, R10 to R15, R11 to R17, R12 to R18, R13 to R20, R14 to R21, R15 to R22, R16 to R23, R17 to R24, R18 to R25, R19 to R26, R20 to R27, R21 to R28, R22 to R29, R2 to R3, R3 to R5, R4 to R7
Connections:
- net GNDA: now also C12.2, C13.2, C17.2, C20.2, C6.2, C9.2, R2.1
- net GNDD: now also R30.1
- net PWM_LPC: now also R2.2
- net at L1.2, R5.2: now also R4.1; no longer U2.1 (IN+)
- net at C10.2, Q1.2 (D), R5.1: now also R6.1; no longer U2.3 (IN-)
- net at C10.1, L2.2: now also D3.2 (A); no longer R9.2, U3.1 (IN+)
- net at C16.1, C18.1, R12.2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: now also R9.1, R11.1, R16.1; no longer D3.1 (K), U5.1 (IN+)
- net at D6.2 (A), R18.1: now also R19.1; no longer U5.3 (IN-)
- net at J4.6 (Shield): now also R30.2
- net L2_current renamed DIODE_current
- net USB_5V renamed VCC
- new net: D3.1 (K), R8.1, R9.2
- new net: C6.1, R4.2, U2.1 (IN+)
- new net: C9.1, R6.2, U2.3 (IN-)
- new net: C17.1, R16.2, U5.1 (IN+)
- new net: C20.1, R19.2, U5.3 (IN-)
- new net: C12.1, R8.2, U3.1 (IN+)
- new net: C13.1, R11.2, U3.3 (IN-)
Other:
- moved on the sheet: C11, C15, C5, D3, L2, R9, U2, U3, U5
